Commit message: Add UR10e XRDF from Isaac Robot Description Editor, re-exported URDF
- AIKIDO.editor.xrdf: editor output (786 spheres incl. gantry frame, vagn,
  wrist camera; spheres in USD link frames)
- AIKIDO.xrdf: same spheres re-based into URDF link frames for cuMotion
  (only the 8 finger links differ) by rebase_xrdf_spheres.py
- AIKIDO.urdf re-exported with the mimic sign fix

File: generative_kitting/robot_config/ur10e/AIKIDO.urdf (robot description, URDF)
Before this commit: robot gantry, 19 links, 18 joints
Joints:
- joint elbow_joint: origin xyz=-0.612699986 -1.83535506e-06 -1.99466833e-08 rpy=8.06233943e-08 -3.25563999e-08 2.99561348e-06 -> xyz=-0.612699986 1.38446415e-06 -2.01023612e-08 rpy=9.31373753e-08 -3.28104676e-08 -2.25968064e-06
- joint finger_joint: origin xyz=3.8417412e-09 -0.0306009073 0.0546625181 rpy=-1.57079633 0 -1.5707962 -> xyz=-1.10565879e-09 -0.0306011457 0.0546625182 rpy=-1.57079633 -1.82875326e-10 -1.57079636
- joint grasp_frame_fixed_joint: origin xyz=0 2.38429913e-07 0.158154975 rpy=0 1.7536907e-10 1.26440403e-07 -> xyz=0 0 0.158154975 rpy=-2.11954905e-10 1.50775151e-10 -4.21460459e-08
- joint left_inner_finger_joint: origin xyz=-0.0354828078 0.0788751575 1.4323272e-08 rpy=9.09204643e-08 2.82666454e-08 0.000666628285 -> xyz=-0.0355057219 0.0788648372 -2.65588017e-08 rpy=-7.22823373e-08 -1.77286225e-08 0.000957323187
- joint left_inner_finger_pad_joint: origin xyz=0.0179063318 0.00650135935 9.63210389e-09 rpy=1.73369589e-07 -3.64109076e-08 -0.000782405366 -> xyz=0.017921698 0.00645796411 -8.60696581e-09 rpy=-1.27295329e-07 -1.27329911e-08 -0.00320146338
- joint left_outer_finger_joint: origin xyz=0.0314311162 0.00448822857 -1.56787868e-08 rpy=4.68598644e-08 -2.11045535e-08 3.14019127 -> xyz=0.0314221386 0.00455084384 2.17017425e-08 rpy=2.71550068e-08 1.38923483e-07 -3.14100456
- joint right_inner_finger_joint: origin xyz=-0.0355182227 0.0788593532 -3.52959731e-09 rpy=3.14159265 -7.69238411e-09 0.00111959513 -> xyz=-0.0355754995 0.0788334797 4.06460044e-08 rpy=-3.14159245 2.39453713e-08 0.00184061717
- joint right_inner_finger_pad_joint: origin xyz=0.0179337737 -0.00642575083 -2.96537378e-08 rpy=-3.14159259 -6.99222907e-08 0.00500231015 -> xyz=0.0179457499 -0.00639145814 1.00667785e-08 rpy=3.14159249 -8.05356316e-09 0.00691528837
- joint right_outer_finger_joint: origin xyz=0.0314266719 0.00452019973 -2.48791659e-08 rpy=-1.52365052e-07 -9.2073987e-08 3.14121019 -> xyz=0.0314225921 0.00454656571 -1.02217176e-08 rpy=-1.32201866e-07 1.54193303e-07 -3.14113842
- joint right_outer_knuckle_joint: mimic joint=finger_joint multiplier=-1 offset=0 -> joint=finger_joint multiplier=1 offset=0; origin xyz=-3.83226179e-09 0.0306013841 0.0546625181 rpy=-1.57079633 0 1.57079645 -> xyz=1.11987991e-09 0.0306011457 0.0546625182 rpy=-1.57079633 1.82875104e-10 1.57079629
- joint shoulder_lift_joint: origin xyz=-5.5753838e-08 1.89410901e-08 -2.9789592e-08 rpy=1.57079624 1.52025749e-08 -0.000481260935 -> xyz=-5.46212733e-08 -5.43409062e-09 -5.95945868e-08 rpy=1.57079623 1.51642689e-08 -0.000424333755
- joint shoulder_pan_joint: origin xyz=4.13463486e-10 -1.32686995e-07 0.18069996 rpy=-1.03206305e-07 -2.52407842e-09 -3.14159257 -> xyz=-3.9980419e-10 -1.36228415e-07 0.180700011 rpy=-9.87895163e-08 2.06467009e-09 -3.14159257
- joint ur10e_gripper_fixed_joint: origin xyz=6.97232343e-08 -2.01030064e-08 -1.4674988e-08 rpy=-1.55206305e-08 -3.560273e-08 -1.57079381 -> xyz=8.72481305e-08 8.04929307e-09 -1.852344e-08 rpy=-1.55040615e-08 -7.91894411e-08 -1.57079531
- joint vagn_robot_joint: origin xyz=-0.0007824963 -1.14684127e-07 -3.7824833e-08 rpy=0 0 0 -> xyz=-0.000767631344 -8.48818047e-08 -6.76271554e-08 rpy=0 0 0
- joint wrist_1_joint: origin xyz=-0.571549964 1.9278736e-06 0.174150322 rpy=0 0 -3.37069404e-06 -> xyz=-0.571549948 2.57202591e-06 0.174150182 rpy=0 0 -4.4943246e-06
- joint wrist_2_joint: origin xyz=-2.47265885e-06 -0.119850006 1.15076331e-07 rpy=1.57079627 4.06120025e-08 -2.1722317e-05 -> xyz=-2.30227668e-06 -0.119849984 1.71844243e-07 rpy=1.57079627 4.08792937e-08 -1.9100657e-05
- joint wrist_3_joint: origin xyz=-3.3166711e-06 0.116550019 -1.84219861e-08 rpy=-1.57079623 -8.73924313e-08 2.70530525e-05 -> xyz=-1.66508748e-06 0.116550042 -1.00841967e-08 rpy=-1.57079616 -8.74236135e-08 1.46938225e-05
